File: varaajamonitori.kicad_pcb (KiCad board)
At the start: 4 copper layers, 105 x 120 mm, 78 parts, among them J1 230Vin, J10 Conn_01x08_Socket, J11 Conn_01x02_Socket, J2 POWER SWITCH, J3 AVR-ISP-6, J4 sensorAAB, J5 SensorBCC, J6 RO1-230VAC-Out, J7 RO2-230VAC-Out, J8 Conn_01x10_Pin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

Commit message: Fixed regulator footprints, removed AC switch
Parts:
- removed J2: POWER SWITCH, Connector_Wire:SolderWire-1.5sqmm_1x04_P6mm_D1.7mm_OD3mm
- removed U5: L7805CV, to254:TO254P1066X482X2286-3
- added U3: L7805CV, varaajamonitori2:TO255P1040X460X1968-3, F.Cu at (141.9, 48.0)
- R5, R6: footprint Resistor_SMD:R_0805_2012Metric_Pad1.20x1.40mm_HandSolder -> Resistor_SMD:R_1206_3216Metric_Pad1.30x1.75mm_HandSolder
- U2: value MIC29510-5.0WT -> L7805CV; footprint to254:TO254P1066X482X2286-3 -> varaajamonitori2:TO255P1040X460X1968-3
- moved U2 6.93 mm to (141.9, 41.5)
- moved D6 1.90 mm to (134.0, 45.7)
Connections:
- F1 pad 2: Net-(J2-Pin_3) -> AC
- J1 pad 2: Net-(J1-Pin_2) -> GNDREF
- U2 pad 1: GND -> /5V1DIRTY
- U2 pad 2: Net-(U2-VO) -> GND
- U2 pad 3: /5V1DIRTY -> +3.3V
Routing:
- net GNDREF: track 77.5 -> 128.4 mm
- net Net-(J1-Pin_2): track 45.4 -> 0.00 mm
- net /driver-M1: track 88.5 -> 114.7 mm
- net VDD: track 245.3 -> 267.5 mm
- net +5V: track 52.4 -> 73.7 mm
- net Net-(U5-VO): track 19.8 -> 0.00 mm
- net GND: track 499.5 -> 480.6 mm
- net Net-(U2-VO): track 16.2 -> 0.00 mm
- net +3.3V: track 73.5 -> 86.7 mm
- net AC: track 27.0 -> 39.5 mm
- net /driver-M2: track 104.9 -> 96.3 mm, vias 1 -> 0
- net /~{RESET}: track 146.9 -> 155.3 mm
- net /MISO: track 99.1 -> 105.2 mm
- net Net-(J2-Pin_3): track 5.47 -> 0.00 mm
- net Net-(D7-A): track 57.6 -> 54.6 mm
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Other:
- board text added: "locked"
- board text removed: "ALAS/(-)"
- board text removed: "DC +3.3V"
- board text removed: "DC +5V"
- board text removed: "Ensiö"
- board text removed: "GND PB2 CS CLK DIN PB0 PB2 D/C M2 M1"
- board text removed: "OIKEA"
- board text removed: "RESETOI"
- board text removed: "TAKAISIN"
- board text removed: "Toisio"
- board text removed: "VALITSE"
- board text removed: "VARAAJAMONITORI"
- board text removed: "VASEN"
- board text removed: "VDD MOSI GND"
- board text removed: "YLÖS/(+)"

Commit message: Changing AC, edge, ACDC
Parts:
- removed C12: C, Capacitor_THT:CP_Radial_D6.3mm_P2.50mm
- removed C13, C14: CP, Capacitor_THT:CP_Radial_D6.3mm_P2.50mm
- removed D6: DZ2S051X0L, Diode_SMD:D_SOD-523
- removed L2: L, Inductor_THT:L_Axial_L5.3mm_D2.2mm_P2.54mm_Vertical_Vishay_IM-1
- removed R2: 1M, Resistor_THT:R_Axial_DIN0309_L9.0mm_D3.2mm_P12.70mm_Horizontal
- removed R4: 5R, Resistor_SMD:R_0805_2012Metric_Pad1.20x1.40mm_HandSolder
- removed R6: 5MR, Resistor_SMD:R_1206_3216Metric_Pad1.30x1.75mm_HandSolder
- removed U2: L7805CV, varaajamonitori2:TO255P1040X460X1968-3
- added Bottom2: Conn_01x01_Pin, varaajamonitori:Drill, F.Cu at (156.6, 146.0)
- added Bottom3: Conn_01x01_Pin, varaajamonitori:Drill, F.Cu at (51.0, 146.2)
- added Bottom4: Conn_01x01_Pin, varaajamonitori:Drill, F.Cu at (103.4, 146.2)
- Bottom1, Mid1: value Conn_01x01_Pin -> locked
- C4: value CP -> 1000uF
- C5: value C -> 10uf
- moved C16 197.4 mm to (236.5, 143.0), turned to 0 degrees
- moved JP2 160.8 mm to (237.2, 134.1), turned to 0 degrees
- moved C4 143.7 mm to (228.4, 136.5), turned to 0 degrees
- moved C7 140.9 mm to (235.6, 103.8)
- moved C5 127.7 mm to (235.6, 88.1), turned to 0 degrees
- moved C6 120.4 mm to (235.6, 96.0)
- moved U3 112.5 mm to (200.9, 143.7)
- moved R19 105.4 mm to (215.6, 111.4)
- moved BZ1 77.6 mm to (21.5, 82.7)
- moved D1 77.6 mm to (14.1, 80.8)
- moved R7 77.6 mm to (24.3, 95.8)
- moved locked 77.6 mm to (31.6, 95.8)
- moved R20 70.1 mm to (215.6, 117.5), turned to 0 degrees
- moved SW2 56.7 mm to (68.5, -11.7)
- moved SW1 56.7 mm to (68.5, -20.4)
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- renumbered Q5 to locked
Connections:
- net Net-(J1-Pin_3) renamed /0-wire
- net Net-(Q3-G) renamed /M1B
- net Net-(Q4-G) renamed /M2B
- net Net-(R17-Pad2) renamed /M1A
- net Net-(R18-Pad2) renamed /M2A
- net Net-(T1-Pad2) renamed /ACT
- C10 pad 2: GNDREF -> /TRIAC AC M1
- C11 pad 2: GNDREF -> /TRIAC AC M2
- J6 pad 2: GNDREF -> /TRIAC AC M1
- J6 pad 3: AC -> GNDREF
- J7 pad 2: GNDREF -> /TRIAC AC M2
- J7 pad 3: AC -> GNDREF
- Q3 pad 1: GNDREF -> /TRIAC AC M1
- Q4 pad 1: GNDREF -> /TRIAC AC M2
- R15 pad 1: GNDREF -> /TRIAC AC M1
- R16 pad 1: GNDREF -> /TRIAC AC M2
Routing:
- net GND: track 480.6 -> 0.00 mm
- net VDD: track 267.5 -> 0.00 mm, vias 1 -> 0
- net /~{RESET}: track 155.3 -> 0.00 mm, vias 1 -> 0
- net GNDREF: track 128.4 -> 0.00 mm
- net /driver-M1: track 114.7 -> 0.00 mm
- net Net-(U1-PC0): track 109.1 -> 0.00 mm, vias 2 -> 0
- net Net-(U1-PC3): track 108.3 -> 0.00 mm, vias 2 -> 0
- net Net-(U1-PC4): track 108.1 -> 0.00 mm, vias 2 -> 0
- net Net-(U1-PC2): track 105.5 -> 0.00 mm, vias 2 -> 0
- net /MISO: track 105.2 -> 0.00 mm, vias 1 -> 0
- net /PB2: track 104.1 -> 0.00 mm
- net /SCK: track 97.9 -> 0.00 mm, vias 1 -> 0
- net Net-(U1-PC1): track 96.9 -> 0.00 mm, vias 2 -> 0
- net /MOSI: track 96.8 -> 0.00 mm, vias 1 -> 0
- net /driver-M2: track 96.3 -> 0.00 mm
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- removed copper zone on In2.Cu, net AC
- removed copper zone on B.Cu, net Earth_Protective
- removed copper zone on F.Cu, net Earth_Protective
- removed copper zone on In1.Cu, net GNDREF
Other:
- board size 105 x 120 mm -> 112.6 x 120 mm
- board text added: "ALAS/(-)"
- board text added: "DC +3.3V"
- board text added: "DC +5V"
- board text added: "Ensiö"
- board text added: "GND PB2 CS CLK DIN PB0 PB2 D/C M2 M1"
- board text added: "OIKEA"
- board text added: "RESETOI"
- board text added: "TAKAISIN"
- board text added: "Toisio"
- board text added: "VALITSE"
- board text added: "VARAAJAMONITORI"
- board text added: "VASEN"
- board text added: "VDD MOSI GND"
- board text added: "YLÖS/(+)"
- board text removed: "locked"

Commit message: New routing tests
Parts:
- removed Bottom2: Conn_01x01_Pin, varaajamonitori:Drill
- removed C3567: CP1_Small, Capacitor_THT:CP_Radial_Tantal_D4.5mm_P5.00mm
- removed C5: 10uf, Capacitor_THT:CP_Radial_D6.3mm_P2.50mm
- removed J10: Conn_01x08_Socket, Connector_PinHeader_2.54mm:PinHeader_1x08_P2.54mm_Vertical
- removed J8: Conn_01x10_Pin, Connector_PinHeader_2.54mm:PinHeader_1x10_P2.54mm_Vertical
- removed R5: 5MR, Resistor_SMD:R_1206_3216Metric_Pad1.30x1.75mm_HandSolder
- removed S1: 452403012014, 452403012014:452403012014
- added C1: 10uf, Capacitor_THT:CP_Radial_D6.3mm_P2.50mm, F.Cu at (146.3, 36.0)
- added C2: 10uf, Capacitor_THT:CP_Radial_D6.3mm_P2.50mm, F.Cu at (52.4, 136.0)
- added C3: 10nF, Capacitor_SMD:C_1206_3216Metric_Pad1.33x1.80mm_HandSolder, F.Cu at (91.4, 140.0)
- added R13: 10kR, Resistor_SMD:R_0805_2012Metric_Pad1.20x1.40mm_HandSolder, F.Cu at (64.4, 90.4)
- added R2: 1MR, Resistor_SMD:R_0805_2012Metric_Pad1.20x1.40mm_HandSolder, F.Cu at (94.4, 136.6)
- added R21: 10kR, Resistor_SMD:R_0805_2012Metric_Pad1.20x1.40mm_HandSolder, F.Cu at (87.0, 90.8)
- added R22: 10kR, Resistor_SMD:R_0805_2012Metric_Pad1.20x1.40mm_HandSolder, F.Cu at (68.4, 93.6)
- added R23: 10kR, Resistor_SMD:R_0805_2012Metric_Pad1.20x1.40mm_HandSolder, F.Cu at (84.2, 75.2)
- added R4: 10kR, Resistor_SMD:R_0805_2012Metric_Pad1.20x1.40mm_HandSolder, F.Cu at (101.4, 84.6)
- added R6: 10kR, Resistor_SMD:R_0805_2012Metric_Pad1.20x1.40mm_HandSolder, F.Cu at (82.8, 91.0)
- added locked: Conn_01x01_Pin, varaajamonitori:Drill, F.Cu at (163.2, 146.0)
- Bottom1, Mid1: value locked -> Conn_01x01_Pin
- C15: value CP1_Small -> 0.1uF; footprint Capacitor_THT:CP_Radial_Tantal_D4.5mm_P5.00mm -> Capacitor_SMD:C_1206_3216Metric_Pad1.33x1.80mm_HandSolder
- C16: value C_Small -> 100nF; footprint Capacitor_THT:C_Disc_D3.0mm_W1.6mm_P2.50mm -> Capacitor_SMD:C_1206_3216Metric_Pad1.33x1.80mm_HandSolder
- C6, C7: value CP -> 1uF
- C8, C9: footprint Capacitor_THT:CP_Radial_Tantal_D4.5mm_P5.00mm -> Capacitor_SMD:C_1206_3216Metric_Pad1.33x1.80mm_HandSolder
- J6: value RO1-230VAC-Out -> RO1-230VAC-PUMP
- J7: value RO2-230VAC-Out -> RO2-230VAC-PUMP
- L1: value L -> 10uH; footprint Inductor_THT:L_Axial_L5.3mm_D2.2mm_P2.54mm_Vertical_Vishay_IM-1 -> Inductor_SMD:L_1206_3216Metric_Pad1.22x1.90mm_HandSolder
- R1: value 5R -> 10kR
- R11, R12, R8, R9: footprint Resistor_SMD:R_0805_2012Metric_Pad1.20x1.40mm_HandSolder -> Resistor_SMD:R_1206_3216Metric_Pad1.30x1.75mm_HandSolder
- R3: value 10kR -> 470R; footprint Resistor_SMD:R_0805_2012Metric_Pad1.20x1.40mm_HandSolder -> Resistor_SMD:R_1206_3216Metric_Pad1.30x1.75mm_HandSolder
- R7: footprint Resistor_THT:R_Axial_DIN0309_L9.0mm_D3.2mm_P12.70mm_Horizontal -> Resistor_SMD:R_0805_2012Metric_Pad1.20x1.40mm_HandSolder
- moved C16 178.1 mm to (58.8, 131.8), turned to -90 degrees
- moved JP2 137.3 mm to (141.0, 36.2)
- moved C4 110.2 mm to (157.9, 51.8)
- moved U3 110.1 mm to (155.6, 43.4), turned to 90 degrees
- moved SW2 104.2 mm to (75.7, 92.2)
- moved SW5 101.1 mm to (75.7, 83.0)
- moved C6 100.7 mm to (148.8, 45.0), turned to 180 degrees
- moved SW3 100.6 mm to (85.0, 83.0)
- moved SW4 100.5 mm to (66.3, 83.0)
- moved C7 100.3 mm to (148.8, 53.6), turned to 180 degrees
- moved R3 98.7 mm to (58.8, 124.6), turned to -90 degrees
- moved SW1 94.1 mm to (76.2, 73.4)
- moved R1 90.6 mm to (63.0, 115.8), turned to 90 degrees
- moved J3 90.6 mm to (51.7, 123.5)
- moved R19 72.9 mm to (142.8, 107.6)
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Connections:
- net Net-(U1-PC0) renamed /UpSw
- net Net-(U1-PC1) renamed /DwnSw
- net Net-(U1-PC2) renamed /RightSw
- net Net-(U1-PC3) renamed /LeftSw
- net Net-(U1-PC4) renamed /SelSw
- net Net-(U1-PC5) renamed /RetSw
- Bottom1 pad 1: GND -> Earth_Protective
- Bottom3 pad 1: GND -> Earth_Protective
- J4 pad 3: GND -> unconnected-(J4-Pin_3-Pad3)
- J5 pad 1: GND -> unconnected-(J5-Pin_1-Pad1)
- JP2 pad 1: +VDC -> +5V
- JP2 pad 3: +BATT -> unconnected-(JP2-B-Pad3)
- Mid1 pad 1: GND -> Earth_Protective
- R1 pad 1: +5V -> Net-(R1-Pad1)
- R1 pad 2: Net-(U2-VO) -> GND
- SW1 pad 2: GND -> Net-(R23-Pad1)
- SW2 pad 2: GND -> Net-(R22-Pad1)
- SW3 pad 2: GND -> Net-(R21-Pad1)
- SW4 pad 2: GND -> Net-(R13-Pad1)
- SW5 pad 2: GND -> Net-(R6-Pad1)
- SW6 pad 2: GND -> Net-(R4-Pad1)
- SW7 pad 2: GND -> Net-(R1-Pad1)
- Top1 pad 1: GND -> Earth_Protective
- Top2 pad 1: GND -> Earth_Protective
- U1 pad 7: GND -> unconnected-(U1-XTAL1/PB6-Pad7)
- U1 pad 8: GND -> unconnected-(U1-XTAL2/PB7-Pad8)
Routing:
- net Earth_Protective: track 0.00 -> 540.6 mm
- net GND: track 0.00 -> 396.7 mm, vias 0 -> 2
- net VDD: track 0.00 -> 251.0 mm
- net AC: track 0.00 -> 120.6 mm
- net GNDREF: track 0.00 -> 89.7 mm
- net /~{RESET}: track 0.00 -> 70.1 mm, vias 0 -> 1
- net /UpSw: track 0.00 -> 68.3 mm, vias 0 -> 2
- net /RightSw: track 0.00 -> 63.1 mm, vias 0 -> 2
- net /RetSw: track 0.00 -> 61.1 mm, vias 0 -> 2
- net /driver-M2: track 0.00 -> 59.0 mm, vias 0 -> 2
- net /LeftSw: track 0.00 -> 56.7 mm, vias 0 -> 2
- net /SelSw: track 0.00 -> 56.2 mm, vias 0 -> 2
- net /TRIAC AC M1: track 0.00 -> 49.1 mm
- net /DwnSw: track 0.00 -> 48.8 mm, vias 0 -> 2
- net /driver-M1: track 0.00 -> 48.7 mm, vias 0 -> 2
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Other:
- board size 112.6 x 120 mm -> 119.8 x 120 mm
- board text removed: "ALAS/(-)"
- board text removed: "DC +3.3V"
- board text removed: "DC +5V"
- board text removed: "Ensiö"
- board text removed: "GND PB2 CS CLK DIN PB0 PB2 D/C M2 M1"
- board text removed: "OIKEA"
- board text removed: "RESETOI"
- board text removed: "TAKAISIN"
- board text removed: "Toisio"
- board text removed: "VALITSE"
- board text removed: "VARAAJAMONITORI"
- board text removed: "VASEN"
- board text removed: "VDD MOSI GND"
- board text removed: "YLÖS/(+)"

Commit message: Adding ISP, UART, I2C plus commenting
Parts:
- added J10: Conn_01x04_Socket, Connector_PinHeader_2.54mm:PinHeader_1x04_P2.54mm_Vertical, F.Cu at (61.4, 66.8)
- added J12: AVR-ISP-6, Connector_PinHeader_2.54mm:PinHeader_2x03_P2.54mm_Vertical, F.Cu at (66.4, 77.0)
- added J13: Conn_01x02_Socket, Connector_PinHeader_2.54mm:PinHeader_1x02_P2.54mm_Vertical, F.Cu at (98.8, 67.5)
- added J14: Conn_01x02_Socket, Connector_PinHeader_2.54mm:PinHeader_1x02_P2.54mm_Vertical, F.Cu at (103.4, 67.5)
- added J2: locked, varaajamonitori:LCD1602 RGB MOD, F.Cu at (91.6, 46.9)
- added J8: AVR-ISP-10, Connector_PinHeader_2.54mm:PinHeader_2x05_P2.54mm_Vertical, F.Cu at (51.7, 66.7)
- added J9: Conn_01x04_Socket, Connector_PinHeader_2.54mm:PinHeader_1x04_P2.54mm_Vertical, F.Cu at (61.4, 71.5)
- added R5: 1000R, Resistor_SMD:R_0805_2012Metric_Pad1.20x1.40mm_HandSolder, F.Cu at (72.8, 136.0)
- R1: footprint Resistor_SMD:R_0805_2012Metric_Pad1.20x1.40mm_HandSolder -> Resistor_SMD:R_1206_3216Metric_Pad1.30x1.75mm_HandSolder
- U1: value ATmega168-20AU -> ATmega328P-P; footprint Package_QFP:TQFP-32_7x7mm_P0.8mm -> Package_DIP:DIP-28_W7.62mm
- moved J11 45.6 mm to (51.7, 86.5), turned to 180 degrees
- moved U1 31.6 mm to (63.4, 95.5), turned to 0 degrees
- moved L1 15.8 mm to (75.2, 132.4), turned to 180 degrees
- moved locked 15.3 mm to (58.4, 84.7)
- moved R7 14.1 mm to (61.8, 91.2)
- moved SW9 13.8 mm to (77.2, 116.4), turned to 90 degrees
- moved R23 9.34 mm to (92.9, 71.8)
- moved R6 9.34 mm to (91.5, 87.6)
- moved SW1 9.34 mm to (84.9, 70.0)
- moved SW2 9.34 mm to (84.4, 88.8)
- moved SW3 9.34 mm to (93.7, 79.6)
- moved SW4 9.34 mm to (75.0, 79.6)
- moved SW5 9.34 mm to (84.4, 79.6)
- moved SW6 9.34 mm to (103.0, 79.6)
- moved R21 9.34 mm to (95.7, 87.4)
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Connections:
- C15 pad 1: Net-(U1-AREF) -> /AVCC
- J4 pad 3: unconnected-(J4-Pin_3-Pad3) -> Net-(J4-Pin_3)
- J5 pad 1: unconnected-(J5-Pin_1-Pad1) -> GND
- L1 pad 2: Net-(U1-AREF) -> /AVCC
- R10 pad 1: VDD -> /AVCC
- R14 pad 1: VDD -> /AVCC
- U1 pad 1: /driver-M2 -> /~{RESET}
- U1 pad 10: /CS -> unconnected-(U1-XTAL2/PB7-Pad10)
- U1 pad 11: /D/C -> /LeftSw
- U1 pad 12: /PB0 -> /SelSw
- U1 pad 13: /PB1 -> /RetSw
- U1 pad 14: /PB2 -> /UpSw
- U1 pad 15: /MOSI -> /DwnSw
- U1 pad 16: /MISO -> /RightSw
- U1 pad 17: /SCK -> /MOSI
- U1 pad 18: Net-(U1-AREF) -> /MISO
- U1 pad 19: /sensor1 -> /SCK
- U1 pad 2: /DIN -> /RX
- U1 pad 20: Net-(U1-AREF) -> /AVCC
- U1 pad 21: GND -> /AVCC
- U1 pad 22: /sensor2 -> GND
- U1 pad 23: /UpSw -> /sensor1
- U1 pad 24: /DwnSw -> /sensor2
- U1 pad 25: /RightSw -> /sensor3
- U1 pad 26: /LeftSw -> /SELA
- U1 pad 27: /SelSw -> /SDA
- U1 pad 28: /RetSw -> /SCL
- U1 pad 3: GND -> /TX
- U1 pad 4: VDD -> /driver-M1
- U1 pad 5: GND -> /driver-M2
- U1 pad 6: VDD -> /SELB
- U1 pad 7: unconnected-(U1-XTAL1/PB6-Pad7) -> VDD
- U1 pad 8: unconnected-(U1-XTAL2/PB7-Pad8) -> GND
- U1 pad 9: /CLK -> unconnected-(U1-XTAL1/PB6-Pad9)
Routing:
- net GND: track 396.7 -> 0.00 mm, vias 2 -> 0
- net VDD: track 251.0 -> 0.00 mm
- net /~{RESET}: track 70.1 -> 0.00 mm, vias 1 -> 0
- net /UpSw: track 68.3 -> 0.00 mm, vias 2 -> 0
- net /RightSw: track 63.1 -> 0.00 mm, vias 2 -> 0
- net /RetSw: track 61.1 -> 0.00 mm, vias 2 -> 0
- net /driver-M2: track 59.0 -> 0.00 mm, vias 2 -> 0
- net /LeftSw: track 56.7 -> 0.00 mm, vias 2 -> 0
- net /SelSw: track 56.2 -> 0.00 mm, vias 2 -> 0
- net /DwnSw: track 48.8 -> 0.00 mm, vias 2 -> 0
- net /driver-M1: track 48.7 -> 0.00 mm, vias 2 -> 0
- net +5V: track 36.7 -> 0.00 mm
- net /PB2: track 33.4 -> 0.00 mm, vias 2 -> 0
- net Net-(U1-AREF): track 28.8 -> 0.00 mm, vias 2 -> 0
- net Net-(D5-AC-Pad2): track 21.6 -> 0.00 mm
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
Commit message: some changes
Parts:
- removed C15: 0.1uF, Capacitor_SMD:C_1206_3216Metric_Pad1.33x1.80mm_HandSolder
- removed D7, D8: LED, LED_THT:LED_D3.0mm
- removed Q1, Q2: BC337, Package_TO_SOT_THT:TO-92_Inline
- removed R8: 470R, Resistor_SMD:R_1206_3216Metric_Pad1.30x1.75mm_HandSolder
- added C13: 100nF, Capacitor_SMD:C_1206_3216Metric_Pad1.33x1.80mm_HandSolder, F.Cu at (67.6, 136.2)
- added C5: 100nF, Capacitor_SMD:C_1206_3216Metric_Pad1.33x1.80mm_HandSolder, F.Cu at (75.6, 100.4)
- added D2: LED, LED_THT:LED_D3.0mm, F.Cu at (70.0, 90.7)
- added D3: 1N4148W-TP, Diode_SMD:D_SOD-123, F.Cu at (53.2, 117.8)
- added D4: LED, LED_THT:LED_D3.0mm, F.Cu at (78.0, 90.5)
- added R24: 390R, Resistor_SMD:R_1206_3216Metric_Pad1.30x1.75mm_HandSolder, F.Cu at (77.2, 84.6)
- BZ1: footprint Buzzer_Beeper:Buzzer_12x9.5RM7.6 -> footprints:CEM-1206S_CUD
- C16: value 100nF -> 1uF
- C8, C9: value CP1_Small -> 100nF
- D1: value 1N4148 -> 1N4148W-TP; footprint Diode_THT:D_DO-35_SOD27_P7.62mm_Horizontal -> Diode_SMD:D_SOD-123
- J4: value sensorAAB -> SensorAAB
- R10, R13, R14, R2, R21, R22, R23, R4, R5, R6: footprint Resistor_SMD:R_0805_2012Metric_Pad1.20x1.40mm_HandSolder -> Resistor_SMD:R_1206_3216Metric_Pad1.30x1.75mm_HandSolder
- R11, R9: value 470R -> 270R
- R12: value 470R -> 390R
- R7: value 330R -> 10kR; footprint Resistor_SMD:R_0805_2012Metric_Pad1.20x1.40mm_HandSolder -> Resistor_SMD:R_1206_3216Metric_Pad1.30x1.75mm_HandSolder
- SW1, SW2, SW3, SW4, SW5, SW6, SW7, SW8, SW9: footprint Button_Switch_SMD:SW_Push_1P1T_NO_CK_KSC6xxJ -> Button_Switch_SMD:SW_Push_1P1T_NO_6x6mm_H9.5mm
- locked: footprint Package_TO_SOT_THT:TO-92_Inline -> Package_TO_SOT_SMD:SOT-23
- moved J14 52.9 mm to (82.9, 116.2), turned to -90 degrees
- moved R12 39.0 mm to (71.2, 84.4), turned to 0 degrees
- moved J13 37.5 mm to (61.7, 73.4)
- moved SW7 35.2 mm to (85.8, 133.7)
- moved locked 22.1 mm to (58.6, 106.8), turned to 0 degrees
- moved R22 20.8 mm to (97.4, 85.5), turned to -90 degrees
- moved R21 19.4 mm to (105.6, 70.8)
- moved R13 19.2 mm to (82.2, 70.2), turned to 90 degrees
- moved L1 18.2 mm to (74.8, 114.2), turned to -90 degrees
- moved R6 18.1 mm to (98.0, 70.8), turned to 0 degrees
- moved C9 17.8 mm to (93.6, 117.8), turned to 180 degrees
- moved C8 13.6 mm to (92.6, 99.4), turned to 180 degrees
- moved R4 10.8 mm to (112.8, 70.8), turned to 180 degrees
- moved J12 10.4 mm to (56.6, 73.4)
- moved J8 10.2 mm to (61.7, 65.1), turned to -90 degrees
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- renumbered Bottom3 to locked
Connections:
- J4 pad 3: Net-(J4-Pin_3) -> /sensor2
- J5 pad 2: /sensor2 -> /sensor3
- R12 pad 1: Net-(R12-Pad1) -> Net-(D2-A)
- R14 pad 2: /sensor2 -> /sensor3
- R5 pad 2: Net-(J4-Pin_3) -> /sensor2
- R9 pad 1: Net-(D8-A) -> Net-(R9-Pad1)
- U6 pad 2: Net-(Q1-C) -> /driver-M1
- U7 pad 1: Net-(R12-Pad1) -> Net-(R9-Pad1)
- U7 pad 2: Net-(Q2-C) -> /driver-M2
Routing:
- net GND: track 0.00 -> 483.7 mm, vias 0 -> 2
- net VDD: track 0.00 -> 306.4 mm
- net /~{RESET}: track 0.00 -> 148.0 mm, vias 0 -> 2
- net /MISO: track 0.00 -> 92.7 mm
- net /RetSw: track 0.00 -> 88.7 mm, vias 0 -> 2
- net /RightSw: track 0.00 -> 87.8 mm, vias 0 -> 2
- net /MOSI: track 0.00 -> 86.1 mm
- net /SCK: track 0.00 -> 85.6 mm, vias 0 -> 1
- net /SelSw: track 0.00 -> 81.8 mm, vias 0 -> 2
- net /UpSw: track 0.00 -> 81.1 mm, vias 0 -> 1
- net /LeftSw: track 0.00 -> 67.5 mm, vias 0 -> 1
- net Net-(R1-Pad1): track 0.00 -> 62.2 mm, vias 0 -> 3
- net /DwnSw: track 0.00 -> 61.3 mm, vias 0 -> 2
- net /driver-M1: track 0.00 -> 56.4 mm, vias 0 -> 1
- net /driver-M2: track 0.00 -> 55.6 mm
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