File: varaajamonitori.kicad_sch (KiCad schematic)
At the start: 78 parts, among them J1 230Vin, J10 Conn_01x08_Socket, J11 Conn_01x02_Socket, J2 POWER SWITCH, J3 AVR-ISP-6, J4 sensorAAB, J5 SensorBCC, J6 RO1-230VAC-Out, J7 RO2-230VAC-Out, J8 Conn_01x10_Pin, Q1 BC337, Q2 BC337, Q3 BT136-500, Q4 BT136-500, Q5 NPN, SW1 UpSw, SW2 DwnSw, SW3 RightSw, SW4 LeftSw, SW5 SelSw, SW6 RetSw, SW7 Reset, SW8 Test1, SW9 Test2, T1 FS12-090-C2, U1 ATmega168-20AU, U2 MIC29510-5.0WT, U5 L7805CV, U6 MOC3020M, U7 MOC3020M

Commit message: Fixed regulator footprints, removed AC switch
Parts:
- removed J2: POWER SWITCH, Connector_Wire:SolderWire-1.5sqmm_1x04_P6mm_D1.7mm_OD3mm, symbol Connector_Generic:Conn_02x02_Odd_Even
- removed R1, R4: 5R, Resistor_SMD:R_0805_2012Metric_Pad1.20x1.40mm_HandSolder, symbol Device:R_Small
- removed U2: MIC29510-5.0WT, to254:TO254P1066X482X2286-3, symbol Regulator_Linear:AP2127N-1.0
- removed U5: L7805CV, to254:TO254P1066X482X2286-3, symbol Regulator_Linear:AP2127N-1.0
- added U2, U3: L7805CV, varaajamonitori2:TO255P1040X460X1968-3, symbol L7805CV:L7805CV
- R5, R6: footprint Resistor_SMD:R_0805_2012Metric_Pad1.20x1.40mm_HandSolder -> Resistor_SMD:R_1206_3216Metric_Pad1.30x1.75mm_HandSolder
Connections:
- net +3.3V: now also U2.3 (OUTPUT)
- net +5V: now also U3.3 (OUTPUT)
- net 5V1DIRTY: now also U2.1 (INPUT), U3.1 (INPUT)
- net AC: now also F1.2
- net GND: now also U2.2 (GROUND), U3.2 (GROUND)
- net GNDREF: now also J1.2 (Pin_2)
Other:
- note removed: "PI3CH281QEX"
- note removed: "~{Select}_ADS1018"

Commit message: Big bug fix to TRIAC
Connections:
- net AC: no longer J6.3 (Pin_3), J7.3 (Pin_3)
- net GNDREF: now also J6.3 (Pin_3), J7.3 (Pin_3); no longer C10.2, C11.2, J6.2 (Pin_2), J7.2 (Pin_2), Q3.1 (A1), Q4.1 (A1), R15.1, R16.1
- new net: C10.2, J6.2 (Pin_2), Q3.1 (A1), R15.1
- new net: C11.2, J7.2 (Pin_2), Q4.1 (A1), R16.1
Changed lines of the file:
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@@
   (junction (at 156.21 68.58) (diameter 0) (color 0 0 0 0)
   )
+  (junction (at 360.68 223.52) (diameter 0) (color 0 0 0 0)
+  )
   (junction (at 342.9 223.52) (diameter 0) (color 0 0 0 0)
   )
@@
   (junction (at 299.72 85.09) (diameter 0) (color 0 0 0 0)
   )
-  (junction (at 360.68 223.52) (diameter 0) (color 0 0 0 0)
-  )
   (junction (at 229.87 153.67) (diameter 0) (color 0 0 0 0)
   )
@@
   (junction (at 176.53 68.58) (diameter 0) (color 0 0 0 0)
   )
+  (junction (at 358.14 166.37) (diameter 0) (color 0 0 0 0)
+  )
   (junction (at 166.37 60.96) (diameter 0) (color 0 0 0 0)
   )
@@
   (junction (at 127 71.12) (diameter 0) (color 0 0 0 0)
   )
-  (junction (at 358.14 166.37) (diameter 0) (color 0 0 0 0)
-  )
   (junction (at 54.61 147.32) (diameter 0) (color 0 0 0 0)
   )
@@
   )
   (no_connect (at 165.1 214.63))
-  (wire (pts (xy 360.68 223.52) (xy 368.3 223.52))
-    (stroke (width 0) (type default))
-  )
   (wire (pts (xy 54.61 147.32) (xy 60.96 147.32))
     (stroke (width 0) (type default))
@@
     (stroke (width 0) (type default))
   )
-  (wire (pts (xy 368.3 213.36) (xy 374.65 213.36))
-    (stroke (width 0) (type default))
-  )
   (wire (pts (xy 128.27 62.23) (xy 128.27 50.8))
     (stroke (width 0) (type default))
@@
     (stroke (width 0) (type default))
   )
+  (wire (pts (xy 358.14 166.37) (xy 372.11 166.37))
+    (stroke (width 0) (type default))
+  )
   (wire (pts (xy 109.22 214.63) (xy 109.22 227.33))
     (stroke (width 0) (type default))
@@
     (stroke (width 0) (type default))
   )
+  (wire (pts (xy 360.68 223.52) (xy 370.84 223.52))
+    (stroke (width 0) (type default))
+  )
   (wire (pts (xy 130.81 60.96) (xy 130.81 68.58))
     (stroke (width 0) (type default))
@@
     (stroke (width 0) (type default))
   )
+  (wire (pts (xy 374.65 158.75) (xy 374.65 166.37))
+    (stroke (width 0) (type default))
+  )
   (wire (pts (xy 140.97 209.55) (xy 165.1 209.55))
     (stroke (width 0) (type default))
@@
     (stroke (width 0) (type default))
   )
-  (wire (pts (xy 370.84 215.9) (xy 374.65 215.9))
-    (stroke (width 0) (type default))
-  )
   (wire (pts (xy 215.9 40.64) (xy 208.28 40.64))
     (stroke (width 0) (type default))
@@
     (stroke (width 0) (type default))
   )
+  (wire (pts (xy 374.65 215.9) (xy 374.65 223.52))
+    (stroke (width 0) (type default))
+  )
   (wire (pts (xy 67.31 180.34) (xy 78.74 180.34))
     (stroke (width 0) (type default))
@@
     (stroke (width 0) (type default))
   )
-  (wire (pts (xy 370.84 140.97) (xy 370.84 158.75))
-    (stroke (width 0) (type default))
-  )
   (wire (pts (xy 90.17 166.37) (xy 90.17 187.96))
     (stroke (width 0) (type default))
@@
     (stroke (width 0) (type default))
   )
-  (wire (pts (xy 370.84 198.12) (xy 370.84 215.9))
+  (wire (pts (xy 372.11 166.37) (xy 372.11 156.21))
     (stroke (width 0) (type default))
   )
@@
     (stroke (width 0) (type default))
   )
+  (wire (pts (xy 370.84 213.36) (xy 374.65 213.36))
+    (stroke (width 0) (type default))
+  )
   (wire (pts (xy 295.91 149.86) (xy 295.91 152.4))
     (stroke (width 0) (type default))
@@
     (stroke (width 0) (type default))
   )
-  (wire (pts (xy 368.3 156.21) (xy 374.65 156.21))
-    (stroke (width 0) (type default))
-  )
   (wire (pts (xy 127 59.69) (xy 118.11 59.69))
     (stroke (width 0) (type default))
@@
     (stroke (width 0) (type default))
   )
+  (wire (pts (xy 372.11 156.21) (xy 374.65 156.21))
+    (stroke (width 0) (type default))
+  )
   (wire (pts (xy 229.87 151.13) (xy 229.87 153.67))
     (stroke (width 0) (type default))
@@
     (stroke (width 0) (type default))
   )
-  (wire (pts (xy 368.3 223.52) (xy 368.3 213.36))
-    (stroke (width 0) (type default))
-  )
   (wire (pts (xy 339.09 217.17) (xy 327.66 217.17))
     (stroke (width 0) (type default))
@@
     (stroke (width 0) (type default))
   )
-  (wire (pts (xy 358.14 140.97) (xy 370.84 140.97))
-    (stroke (width 0) (type default))
-  )
   (wire (pts (xy 92.71 179.07) (xy 92.71 190.5))
     (stroke (width 0) (type default))
@@
     (stroke (width 0) (type default))
   )
-  (wire (pts (xy 360.68 198.12) (xy 370.84 198.12))
-    (stroke (width 0) (type default))
-  )
   (wire (pts (xy 285.75 80.01) (xy 303.53 80.01))
     (stroke (width 0) (type default))
@@
     (stroke (width 0) (type default))
   )
-  (wire (pts (xy 370.84 158.75) (xy 374.65 158.75))
-    (stroke (width 0) (type default))
-  )
   (wire (pts (xy 336.55 160.02) (xy 327.66 160.02))
     (stroke (width 0) (type default))
@@
     (stroke (width 0) (type default))
   )
-  (wire (pts (xy 368.3 166.37) (xy 368.3 156.21))
-    (stroke (width 0) (type default))
-  )
   (wire (pts (xy 295.91 233.68) (xy 308.61 233.68))
     (stroke (width 0) (type default))
@@
     (stroke (width 0) (type default))
   )
-  (wire (pts (xy 358.14 166.37) (xy 368.3 166.37))
+  (wire (pts (xy 370.84 223.52) (xy 370.84 213.36))
     (stroke (width 0) (type default))
   )
@@
     )
   )
-  (symbol (lib_id "power:GNDREF") (at 358.14 166.37 0) (unit 1)
-    (in_bom yes) (on_board yes) (dnp no)
-    (property "Reference" "#PWR039" (at 358.14 172.72 0)
-      (effects (font (size 1.27 1.27)) hide)
-    )
-    (property "Value" "GNDREF" (at 358.267 170.7642 0)
-      (effects (font (size 1.27 1.27)))
-    )
-    (property "Footprint" "" (at 358.14 166.37 0)
-      (effects (font (size 1.27 1.27)) hide)
-    )
-    (property "Datasheet" "" (at 358.14 166.37 0)
-      (effects (font (size 1.27 1.27)) hide)
-    )
-    (pin "1")
-    (instances
-      (project "varaajamonitori"
-        (path "/f130c31c-315f-477b-9a38-5a4be0e8af48"
-          (reference "#PWR039") (unit 1)
-        )
-      )
-    )
-  )
   (symbol (lib_id "Relay_SolidState:MOC3020M") (at 320.04 152.4 0) (unit 1)
     (in_bom yes) (on_board yes) (dnp no)
@@
     )
   )
-  (symbol (lib_id "power:GNDREF") (at 360.68 223.52 0) (unit 1)
+  (symbol (lib_id "power:GNDREF") (at 374.65 223.52 0) (unit 1)
     (in_bom yes) (on_board yes) (dnp no)
-    (property "Reference" "#PWR041" (at 360.68 229.87 0)
+    (property "Reference" "#PWR041" (at 374.65 229.87 0)
       (effects (font (size 1.27 1.27)) hide)
     )
-    (property "Value" "GNDREF" (at 360.807 227.9142 0)
+    (property "Value" "GNDREF" (at 374.777 227.9142 0)
       (effects (font (size 1.27 1.27)))
     )
-    (property "Footprint" "" (at 360.68 223.52 0)
+    (property "Footprint" "" (at 374.65 223.52 0)
       (effects (font (size 1.27 1.27)) hide)
     )
-    (property "Datasheet" "" (at 360.68 223.52 0)
+    (property "Datasheet" "" (at 374.65 223.52 0)
       (effects (font (size 1.27 1.27)) hide)
     )
@@
         )
       )
+    )
+  )
+  (symbol (lib_id "power:GNDREF") (at 374.65 166.37 0) (unit 1)
+    (in_bom yes) (on_board yes) (dnp no)
+    (property "Reference" "#PWR013" (at 374.65 172.72 0)
+      (effects (font (size 1.27 1.27)) hide)
+    )
+    (property "Value" "GNDREF" (at 374.777 170.7642 0)
+      (effects (font (size 1.27 1.27)))
+    )
+    (property "Footprint" "" (at 374.65 166.37 0)
+      (effects (font (size 1.27 1.27)) hide)
+    )
+    (property "Datasheet" "" (at 374.65 166.37 0)
+      (effects (font (size 1.27 1.27)) hide)
+    )
+    (pin "1")
+    (instances
+      (project "varaajamonitori"
+        (path "/f130c31c-315f-477b-9a38-5a4be0e8af48"
+          (reference "#PWR013") (unit 1)
+        )
+      )

Commit message: Changing AC, edge, ACDC
Parts:
- removed C12: C, Capacitor_THT:CP_Radial_D6.3mm_P2.50mm, symbol Device:C
- removed C13, C14: CP, Capacitor_THT:CP_Radial_D6.3mm_P2.50mm, symbol varaajamonitori-rescue:CP-Device
- removed D6: DZ2S051X0L, Diode_SMD:D_SOD-523, symbol Diode:DZ2S051X0L
- removed L2: L, Inductor_THT:L_Axial_L5.3mm_D2.2mm_P2.54mm_Vertical_Vishay_IM-1, symbol Device:L
- removed R2: 1M, Resistor_THT:R_Axial_DIN0309_L9.0mm_D3.2mm_P12.70mm_Horizontal, symbol Device:R
- removed R6: 5MR, Resistor_SMD:R_1206_3216Metric_Pad1.30x1.75mm_HandSolder, symbol Device:R_Small
- removed S1: 452403012014, 452403012014:452403012014, symbol 452403012014:452403012014
- removed U2: L7805CV, varaajamonitori2:TO255P1040X460X1968-3, symbol L7805CV:L7805CV
- added Bottom2, Bottom3, Bottom4: Conn_01x01_Pin, varaajamonitori:Drill, symbol Connector:Conn_01x01_Pin
- C4: value CP -> 1000uF
- C5: value C -> 10uf
Connections:
- net +VDC is gone; now on net +5V: JP2.1 (A)
- net Earth_Protective: now also Bottom2.1 (Pin_1), Bottom4.1 (Pin_1)
- net GND: now also Bottom3.1 (Pin_1)
- net 0-wire: now reaches F1.1, J1.3 (Pin_3)
- net TRIAC AC M1: now reaches C10.2, J6.2 (Pin_2), Q3.1 (A1), R15.1
- net M1A: now reaches R17.2, U6.6
- net M1B: now reaches Q3.3 (G), R15.2, U6.4
- net M2B: now reaches Q4.3 (G), R16.2, U7.4
- net M2A: now reaches R18.2, U7.6
- net TRIAC AC M2: now reaches C11.2, J7.2 (Pin_2), Q4.1 (A1), R16.1
- net ACT: now reaches T1.2, T1.3
- net +BATT: no longer names the net of JP2.3 (B)
- no-connect marks 1 -> 2
Other:
- note removed: "Select voltage level"
- moved on the sheet: C5

Commit message: New routing tests
Parts:
- removed C3567: CP1_Small, Capacitor_THT:CP_Radial_Tantal_D4.5mm_P5.00mm, symbol varaajamonitori-rescue:CP1_Small-Device
- removed C5: 10uf, Capacitor_THT:CP_Radial_D6.3mm_P2.50mm, symbol Device:C
- removed J10: Conn_01x08_Socket, Connector_PinHeader_2.54mm:PinHeader_1x08_P2.54mm_Vertical, symbol Connector:Conn_01x08_Socket
- removed J8: Conn_01x10_Pin, Connector_PinHeader_2.54mm:PinHeader_1x10_P2.54mm_Vertical, symbol Connector:Conn_01x10_Pin
- added C1, C2: 10uf, Capacitor_THT:CP_Radial_D6.3mm_P2.50mm, symbol varaajamonitori-rescue:CP-Device
- added C3: 10nF, Capacitor_THT:CP_Radial_Tantal_D4.5mm_P5.00mm, symbol varaajamonitori-rescue:CP1_Small-Device
- added R1, R13, R21, R22, R23, R4, R6: 10kR, Resistor_THT:R_Axial_DIN0309_L9.0mm_D3.2mm_P12.70mm_Horizontal, symbol Device:R_Small
- added R2: 1MR, Resistor_SMD:R_0805_2012Metric_Pad1.20x1.40mm_HandSolder, symbol Device:R_Small
- C15: value CP1_Small -> 0.1uF
- J6: value RO1-230VAC-Out -> RO1-230VAC-PUMP
- J7: value RO2-230VAC-Out -> RO2-230VAC-PUMP
- L1: value L -> 10uH
- R3: value 10kR -> 470R
Connections:
- net +5V: now also C1.1
- net Earth_Protective: now also Bottom1.1 (Pin_1), Bottom3.1 (Pin_1), Mid1.1 (Pin_1), Top1.1 (Pin_1), Top2.1 (Pin_1)
- net GND: now also C1.2, C2.2, C3.1, R1.2, R13.2, R2.2, R21.2, R22.2, R23.2, R4.2, R6.2; no longer Bottom1.1 (Pin_1), Bottom3.1 (Pin_1), J4.3 (Pin_3), J5.1 (Pin_1), Mid1.1 (Pin_1), SW1.2, SW2.2, SW3.2, SW4.2, SW5.2, SW6.2, SW7.2, Top1.1 (Pin_1), Top2.1 (Pin_1), U1.7 (XTAL1/PB6), U1.8 (XTAL2/PB7)
- net GNDREF: now also C3.2, R2.1
- net VDD: now also C2.1
- net UpSw: now reaches SW1.1, U1.23 (PC0)
- net DwnSw: now reaches SW2.1, U1.24 (PC1)
- net RightSw: now reaches SW3.1, U1.25 (PC2)
- net LeftSw: now reaches SW4.1, U1.26 (PC3)
- net SelSw: now reaches SW5.1, U1.27 (PC4)
- net RetSw: now reaches SW6.1, U1.28 (PC5)
- new net: R4.1, SW6.2
- new net: R23.1, SW1.2
- new net: R13.1, SW4.2
- new net: R21.1, SW3.2
- new net: R6.1, SW5.2
- new net: R22.1, SW2.2
- new net: R1.1, SW7.2
- no-connect marks 2 -> 5
Other:
- note added: "Bypass cap to remove noise"
- note added: "Inductor isolates AVCC and AREF from VDD"
- note added: "Triac to turn on pump #1"
- note added: "Triac to turn on pump #2"
- note removed: "TPS62750DSKT"
- moved on the sheet: BZ1, C15, C16, D1, L1, Q5, R3, R7, SW1, SW2, SW3, SW4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
